File: single_board/BME688_Breakout_Board.kicad_pcb (KiCad board)
At the start: 4 copper layers, 26 x 19 mm, 19 parts, among them J1 External, Q1 BSS138, Q2 BSS138, Q3 BSS138, U1 BME688, U2 STLQ020C33R

Commit message: Added project libs
Parts:
- added C3: 100n, Capacitor_SMD:C_0402_1005Metric, F.Cu at (223.8, 122.6)
- added C4: 100n, Capacitor_SMD:C_0402_1005Metric, F.Cu at (224.3, 121.1)
- U2: footprint SamacSys_Parts:SOT65P210X110-5N -> BME688_Breakout_Board:SOT323-5L
- moved C1 3.57 mm to (216.5, 129.4), turned to 0 degrees
- moved C2 0.58 mm to (216.3, 124.0)
Routing:
- net VCC: track 43.7 -> 37.8 mm, vias 2 -> 1
- net GND: track 16.2 -> 18.6 mm
- net /+3.3V_SDO: track 19.9 -> 21.6 mm
- net +3V3: track 19.7 -> 18.4 mm, vias 7 -> 8
Other:
- board text added: "Rev. 2.0"
- board text removed: "Rev. 1.5"
