File: single_board/BME688_Breakout_Board.kicad_sch (KiCad schematic)
At the start: 17 parts, among them J1 External, Q1 BSS138, Q2 BSS138, Q3 BSS138, U1 BME688, U2 STLQ020C33R

Commit message: Added project libs
Parts:
- added C3: 100n, Capacitor_SMD:C_0402_1005Metric, symbol Device:C_Small
- added C4: (no value), Capacitor_SMD:C_0402_1005Metric, symbol Device:C_Small
- Q3: value BSS138 -> (none); footprint Package_TO_SOT_SMD:SOT-23 -> (none)
- U1: value BME688 -> (none); symbol BHIT_KiCAD_Library:BME688 -> BME688_Breakout_Board:BME688
- U2: value STLQ020C33R -> (none); footprint SamacSys_Parts:SOT65P210X110-5N -> (none); symbol SamacSys_Parts:STLQ020J33R -> BME688_Breakout_Board:STLQ020C33R
Connections:
- net +3V3: now also C3.1, C4.1
- net GND: now also C3.2, C4.2
Other:
- moved on the sheet: C1, C2, D1, U1
