File: panel/BME688_Breakout_Board_Panel.kicad_pcb (KiCad board)
At the start: 4 copper layers, 100 x 100 mm, 549 parts, among them J1 External, Q1 BSS138, Q2 BSS138, Q3 BSS138, U1 BME688, U2 STLQ020C33R

Commit message: Added project libs
Parts:
- U2 (x12): footprint SamacSys_Parts:SOT65P210X110-5N -> BME688 Footprints:SOT323-5L

Commit message: Corrections
Other:
- board text added: "100.0000 mm x 100.0000 mm"
- board text added: "Bosch Sensortec BME688 Breakout Boards"
- board text added: "Dielectric"
- board text added: "Purple"
- board text added: "Rev. 1.6"
- board text added: "White"
- board text removed: "100.0500 mm x 100.0500 mm"
- board text removed: "3.3V < VCC & Logic< 5V"
- board text removed: "BME280"
- board text removed: "BME280 Barometric Sensor -Pressure -Humidity -Temperature 3.3V < VCC & Logic< 5V"
- board text removed: "BME680"
- board text removed: "BME680 Air Quality Sensor -Pressure -Humidity -Temperature -VOC & eCO2 3.3V < VCC & Logic< 5V"
- board text removed: "BST Sensors Breakout Boards"
- board text removed: "Bosch Sensortec Sensor Breakout Boards"
- board text removed: "Dielectric 1"
- board text removed: "Dielectric 2"
- board text removed: "Dielectric 3"
- board text removed: "Rev. 1.5"
